File: dice-roller-pcb/dice-roller-pcb.kicad_pcb (KiCad board)
At the start: 2 copper layers, 56 x 94.5 mm, 53 parts, among them J1 Conn_01x04_Pin, J2 Conn_01x02_Socket, Q1 AO3400, Q2 AO3400, Q3 AO3400, U1 ESP-12F, U2 RT9013-33GB

Commit message: Update repository
Connections:
- OLED1 pad 5: /OLED_RES -> +3.3V
Routing:
- net +3.3V: track 71.7 -> 74.7 mm
