File: dice-roller-pcb/dice-roller-pcb.kicad_sch (KiCad schematic)
At the start: 47 parts, among them J1 Conn_01x04_Pin, J2 Conn_01x02_Socket, Q1 AO3400, Q2 AO3400, Q3 AO3400, U1 ESP-12F, U2 RT9013-33GB

Commit message: Update repository
Parts:
- M1, OLED1: value ~ -> (none)
Connections:
- net +3.3V: now also OLED1.5 (RES)
- no-connect marks 10 -> 9
